File: bee-pow.kicad_pcb (KiCad board)
At the start: 2 copper layers, 29 x 53.3 mm, 41 parts, among them J1 Conn_01x02_Male, J2 Conn_01x02_Male, J3 Conn_01x02_Male, J4 Conn_01x02_Male, J5 Screw_Terminal_01x03, J6 Screw_Terminal_01x02, U1 L7805, U2 L7815, U3 L7915

Commit message: schematic and layout
Parts:
- removed D10, D12, D15: 1N4001, Diode_THT:D_A-405_P12.70mm_Horizontal
- removed D4, D7, D8: D_Schottky, Diode_THT:D_A-405_P10.16mm_Horizontal
- removed J6: Screw_Terminal_01x02, TerminalBlock:TerminalBlock_bornier-2_P5.08mm
- C1, C2, C3, C5, C6, D11, D13, D14: moved to F.Cu
- C7, C8, C9: footprint Capacitor_THT:CP_Radial_D10.0mm_P5.00mm -> Capacitor_THT:CP_Radial_D8.0mm_P2.50mm
- J5: value Screw_Terminal_01x03 -> Screw_Terminal_01x04; footprint TerminalBlock:TerminalBlock_bornier-3_P5.08mm -> TerminalBlock:TerminalBlock_bornier-4_P5.08mm
- moved C4 96.3 mm to (88.4, 138.2), turned to 90 degrees
- moved D18 85.0 mm to (88.4, 113.8), turned to 90 degrees
- moved C1 84.6 mm to (88.4, 131.1), turned to 270 degrees
- moved D1 84.5 mm to (95.5, 91.4)
- moved R1 84.5 mm to (90.4, 91.4)
- moved R2 78.0 mm to (90.4, 94.0)
- moved D2 77.0 mm to (95.5, 94.0)
- moved C7 76.9 mm to (99.1, 126.0), turned to 90 degrees
- moved C3 75.9 mm to (88.4, 110.2), turned to 90 degrees
- moved C9 63.5 mm to (99.1, 116.8), turned to 90 degrees
- moved D11 58.3 mm to (91.7, 134.6), turned to 270 degrees
- moved D16 57.6 mm to (88.4, 134.6), turned to 90 degrees
- moved U1 57.5 mm to (84.8, 132.1), turned to 270 degrees
- moved U3 54.2 mm to (91.9, 116.3), turned to 90 degrees
- moved C6 41.3 mm to (88.4, 117.3), turned to 90 degrees
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Connections:
- D2 pad 1: GND -> Net-(D2-Pad1)
- D2 pad 2: Net-(D2-Pad2) -> GND
- J5 pad 2: GND -> U2
- J5 pad 3: U2 -> U3
- JP1 pad 1: U3 -> U3_1
- JP2 pad 3: U3 -> U3_1
- R2 pad 2: Net-(D2-Pad2) -> Net-(D2-Pad1)
Routing:
- net U_B+: track 0.00 -> 92.8 mm, vias 0 -> 1
- net U_B-: track 0.00 -> 69.5 mm, vias 0 -> 1
- net U_B2: track 0.00 -> 63.4 mm
- net GND: track 0.00 -> 31.4 mm, vias 0 -> 4
- net Net-(D9-Pad2): track 0.00 -> 17.3 mm
- net Net-(C1-Pad1): track 0.00 -> 15.7 mm, vias 0 -> 1
- net Net-(C2-Pad1): track 0.00 -> 15.5 mm, vias 0 -> 1
- net U3: track 0.00 -> 12.9 mm
- net U1: track 0.00 -> 12.8 mm
- net Net-(C3-Pad2): track 0.00 -> 11.6 mm
- net U2: track 0.00 -> 7.45 mm
- net U3_1: track 0.00 -> 3.56 mm
- net Net-(D2-Pad1): track 0.00 -> 3.05 mm
- net Net-(D1-Pad2): track 0.00 -> 3.03 mm
- net Net-(D3-Pad2): track 0.00 -> 2.54 mm
- added copper zone on B.Cu, net GND
